File: KiCad/FreeEEG32-alpha2.kicad_pcb (KiCad board)
At the start: 4 copper layers, 66 x 66 mm, 192 parts, among them J1 CONN_01X02, J2 USB_C_Receptacle, J3 Conn_02x02_Odd_Even, P1 CONN_02X10, P11 CONN_01X03, P2 CONN_02X10, P3 CONN_02X10, P4 CONN_02X10, P5 USB_OTG, P6 CONN_02X03, P7 CONN_02X03, SW1 NRST, SW2 BOOT0, SW3 RST, SW4 BOOT, T1 da2303, U1 ADP7118AUJZ-3.3, U10 ISO7341c_spi, U11 AMS1117-3.3, U12 LSM6DS3, U13 AD7770, U2 ADP7118AUJZ-3.3, U20 AD7770, U27 AD7770, U3 8.192MHz, U34 AD7770, U37 STM32F427ZI_4side_short, U4 ADR4525, U43 473521001, U5 ADUM1402BRWZ, U6 SN6505B, U7 ESP32-WROOM-32, U8 CP2102N-28, U9 ADUM1402BRWZ, Y1 32768Hz, Y2 8MHz

Commit message: Add files via upload
Parts:
- removed D3: SP0503BAHTG, Package_TO_SOT_SMD:SOT-143
- removed the H4 at (27.9, 27.9)
- removed J3: Conn_02x02_Odd_Even, Connector_PinHeader_2.54mm:PinHeader_2x02_P2.54mm_Horizontal
- removed P11: CONN_01X03, Connector_PinSocket_2.54mm:PinSocket_1x03_P2.54mm_Vertical
- removed P5: USB_OTG, Connector_USB:USB_Micro-B_Molex-105017-0001
- removed REF**: USB_Micro-B_Wuerth_629105150521_CircularHoles, Connector_USB:USB_Micro-B_Wuerth_629105150521_CircularHoles
- added C139: 100n, Capacitor_SMD:C_0402_1005Metric, F.Cu at (74.5, 21.1)
- added C140: 100n, Capacitor_SMD:C_0402_1005Metric, F.Cu at (67.0, 26.5)
- added C141: 1u, Capacitor_SMD:C_0402_1005Metric, B.Cu at (-4.45, 37.7)
- added C142: 1u, Capacitor_SMD:C_0402_1005Metric, B.Cu at (-15.1, 28.3)
- added H4: MountingHole, MountingHole:MountingHole_2.7mm_M2.5_ISO14580_Pad, F.Cu at (29.2, 33.0)
- added H4: MountingHole, MountingHole:MountingHole_2.7mm_M2.5_ISO14580_Pad, F.Cu at (-29.2, 33.0)
- added H4: MountingHole, MountingHole:MountingHole_2.7mm_M2.5_ISO14580_Pad, F.Cu at (-29.2, 10.2)
- added H4: MountingHole, MountingHole:MountingHole_2.7mm_M2.5_ISO14580_Pad, F.Cu at (29.2, 10.2)
- added J10: Conn_01x02, Connector_PinHeader_2.54mm:PinHeader_1x02_P2.54mm_Vertical, F.Cu at (-4.45, 5.08)
- added J11: USB_C_Receptacle-Connector_VBUS2, Connector_USB:USB_C_Receptacle_Amphenol_12401548E4-2A, B.Cu at (19.7, 33.7)
- added J12: Conn_01x02, Connector_PinHeader_2.54mm:PinHeader_1x02_P2.54mm_Vertical, F.Cu at (-9.53, 2.54)
- added J4: Conn_02x07_Odd_Even, Connector_PinSocket_2.54mm:PinSocket_2x07_P2.54mm_Horizontal, F.Cu at (26.7, 29.2)
- added J5: Conn_01x02, Connector_PinHeader_2.54mm:PinHeader_1x02_P2.54mm_Vertical, F.Cu at (12.1, 5.08)
- added J6: Conn_02x20_Odd_Even, Connector_PinSocket_2.54mm:PinSocket_2x20_P2.54mm_Vertical, F.Cu at (24.1, 11.4)
- added J7: Conn_01x02, Connector_PinHeader_2.54mm:PinHeader_1x02_P2.54mm_Vertical, F.Cu at (6.99, 5.08)
- added J8: Conn_01x02, Connector_PinHeader_2.54mm:PinHeader_1x02_P2.54mm_Vertical, F.Cu at (12.1, -5.08)
- added J9: Conn_01x02, Connector_PinHeader_2.54mm:PinHeader_1x02_P2.54mm_Vertical, F.Cu at (6.99, -5.08)
- added P8: USB_OTG, Connector_USB:USB_Micro-B_Molex-105017-0001, F.Cu at (52.4, 57.8)
- added R10: 0, Resistor_SMD:R_0402_1005Metric, F.Cu at (-43.5, 24.5)
- added U14: ISO7341c_spi, Package_SO:SOIC-16W_7.5x10.3mm_P1.27mm, F.Cu at (71.7, 15.1)
- added U15: ISO7341c_spi, Package_SO:SOIC-16W_7.5x10.3mm_P1.27mm, F.Cu at (83.1, 15.1)
- added U16: ISO7341c_spi, Package_SO:SOIC-16W_7.5x10.3mm_P1.27mm, F.Cu at (94.4, 15.1)
- added U17: CAT24M01W, Package_SO:SOIC-8_3.9x4.9mm_P1.27mm, F.Cu at (69.8, 23.3)
- C109, C110, C117, C121, C129, C131, C3, C4, R1, U11: moved to F.Cu
- C125, C133, C136, C138, D4, R6, R9, SW1, SW3: moved to B.Cu
- H1, H3: footprint MountingHole:MountingHole_2.2mm_M2_ISO7380_Pad -> MountingHole:MountingHole_2.7mm_M2.5_ISO14580_Pad
- J1: value CONN_01X02 -> Conn_02x07_Odd_Even; footprint Connector_PinSocket_2.54mm:PinSocket_1x02_P2.54mm_Vertical -> Connector_PinSocket_2.54mm:PinSocket_2x07_P2.54mm_Horizontal
- J2: value USB_C_Receptacle -> USB_C_Receptacle-Connector_VBUS2; footprint Connector_USB:USB_C_Receptacle_Amphenol_12401610E4-2A_CircularHoles -> Connector_USB:USB_C_Receptacle_Amphenol_12401548E4-2A; moved to B.Cu
- P6, P7: value CONN_02X03 -> USB_OTG; footprint Connector_PinSocket_2.54mm:PinSocket_2x03_P2.54mm_Vertical -> Connector_USB:USB_Micro-B_Molex-105017-0001
- T1: footprint da2303:da2303 -> 750315371:750315371
- U12: footprint Housings_LGA_FreeEEG32:LGA-14L_2.5x3mm_Pitch0.5mm -> LSM6DS3TR:Bosch_LGA-14_3x2.5mm_P0.5mm
- U3: footprint Crystal:Crystal_SMD_7050-4Pin_7.0x5.0mm -> Oscillator_Oscillator_SMD_EuroQuartz_XO91-4Pin_7.0x5:Oscillator_SMD_EuroQuartz_XO91-4Pin_7.0x5.0mm_HandSoldering
- Y1: footprint Crystal:Crystal_SMD_MicroCrystal_CC4V-T1A-2Pin_5.0x1.9mm -> Crystal:Crystal_SMD_EuroQuartz_EQ161-2Pin_3.2x1.5mm_HandSoldering; moved to F.Cu
- Y2: footprint Crystal:Crystal_SMD_5032-4Pin_5.0x3.2mm -> smd5032:Crystal_SMD_EuroQuartz_MJ-4Pin_5.0x3.2mm_HandSoldering; moved to F.Cu
- moved P7 139.8 mm to (91.3, 38.7)
- moved H2 121.2 mm to (91.6, 47.9)
- moved P6 95.3 mm to (43.5, 57.8)
- moved R8 45.5 mm to (23.5, 16.5), turned to 180 degrees
- moved C133 41.1 mm to (-17.8, 22.9), turned to 180 degrees
- moved J2 39.9 mm to (-18.8, 33.7), turned to 180 degrees
- moved C136 34.0 mm to (-15.2, 24.1), turned to 180 degrees
- moved R9 33.4 mm to (-14.6, 21.1), turned to 90 degrees
- moved C4 31.1 mm to (7.62, 14.6), turned to 270 degrees
- moved R1 28.0 mm to (6.35, 14.6), turned to 270 degrees
- moved C137 25.8 mm to (10.2, 35.6), turned to 270 degrees
- moved Y2 23.9 mm to (2.54, 15.9)
- moved C135 19.9 mm to (11.4, 35.6)
- moved C131 18.5 mm to (-3.17, 14.6), turned to 270 degrees
- moved C138 18.2 mm to (-17.8, 24.1), turned to 180 degrees
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Connections:
- net IO0_WIFI renamed GPIO0_WIFI
- net Net-(R2-Pad2) renamed BOOT0
- net Net-(R3-Pad1) renamed BOOT1
- net Net-(U37-Pad22) renamed AD_DRDY
- net Net-(U7-Pad24) renamed GPIO2_WIFI
- net SPI4_MISO renamed Net-(U37-Pad4)
- net SPI4_MOSI renamed AD1_DOUT1_ISO
- net SPI6_MOSI renamed Net-(U37-Pad129)
- C1 pad 1: GND_USB -> GND_PWRrt1_USB_C
- C1 pad 2: VDD -> 3V3_RPi
- C10 pad 1: GND_USB -> GND_PWRrt1_USB_C
- C10 pad 2: VDD -> 3V3_RPi
- C100 pad 1: GND_USB -> GND_PWRrt1_USB_C
- C100 pad 2: VDD -> 3V3_RPi
- C101 pad 1: GND_USB -> GND_PWRrt1_USB_C
- C101 pad 2: VDD -> 3V3_RPi
- C102 pad 2: GND_USB -> GND_PWRrt1_USB_C
- C103 pad 1: GND_USB -> GND_PWRrt1_USB_C
- C103 pad 2: VDD -> 3V3_RPi
- C104 pad 1: GND_USB -> GND_PWRrt1_USB_C
- C104 pad 2: VDD -> 3V3_RPi
- C105 pad 1: GND_USB -> GND_PWRrt1_USB_C
- C105 pad 2: VDD -> 3V3_RPi
- C106 pad 1: GND_USB -> GND_PWRrt1_USB_C
- C106 pad 2: VDD -> 3V3_RPi
- C107 pad 1: VDD -> 3V3_RPi
- C107 pad 2: GND_USB -> GND_PWRrt1_USB_C
- C108 pad 1: VDD -> 3V3_RPi
- C108 pad 2: GND_USB -> GND_PWRrt1_USB_C
- C109 pad 1: V+ -> 5V_RPi
- C109 pad 2: GND_USB -> GND_PWRrt1_USB_C
- C11 pad 1: GND_USB -> GND_PWRrt1_USB_C
- C11 pad 2: VDD -> 3V3_RPi
- C110 pad 1: VDD -> 3V3_RPi
- C110 pad 2: GND_USB -> GND_PWRrt1_USB_C
- C114 pad 1: AD1_START -> GND_ISO_RAW
- C114 pad 2: V+_ISO -> V+_ISO_RAW
- C115 pad 1: AD1_START -> GND_ISO_RAW
- C115 pad 2: V+_ISO -> V+_ISO_RAW
- C116 pad 1: GND_USB -> GND_PWRrt1_USB_C
- C116 pad 2: VDD -> 3V3_RPi
- C117 pad 1: V+ -> 5V_RPi
- C117 pad 2: GND_USB -> GND_PWRrt1_USB_C
- C118 pad 1: GND_USB -> GND_PWRrt1_USB_C
- C118 pad 2: VDD -> 3V3_RPi
- C121 pad 1: VDD -> 3V3_RPi
- C121 pad 2: GND_USB -> GND_PWRrt1_USB_C
- C124 pad 2: GND_USB -> GND_PWRrt1_USB_C
- C125 pad 1: GND_USB -> GND_PWRrt1_USB_C
- C128 pad 1: VDD -> 3V3_RPi
- C128 pad 2: GND_USB -> GND_PWRrt1_USB_C
- C129 pad 2: GND_USB -> GND_PWRrt1_USB_C
- C130 pad 1: VDD -> 3V3_RPi
- C130 pad 2: GND_USB -> GND_PWRrt1_USB_C
- C131 pad 2: GND_USB -> GND_PWRrt1_USB_C
- C132 pad 1: VDD -> 3V3_RPi
- C132 pad 2: GND_USB -> GND_PWRrt1_USB_C
- C133 pad 2: GND_USB -> GND_PWRrt1_USB_C
- C134 pad 1: VDD -> 3V3_RPi
- C134 pad 2: GND_USB -> GND_PWRrt1_USB_C
- C135 pad 1: VDD -> 3V3_RPi
- C135 pad 2: GND_USB -> GND_PWRrt1_USB_C
- C136 pad 2: GND_USB -> GND_PWRrt1_USB_C
- C137 pad 1: VDD -> 3V3_RPi
- C137 pad 2: GND_USB -> GND_PWRrt1_USB_C
- C138 pad 2: GND_USB -> GND_PWRrt1_USB_C
- C2 pad 1: GND_USB -> GND_PWRrt1_USB_C
- C2 pad 2: VDD -> 3V3_RPi
- C3 pad 2: GND_USB -> GND_PWRrt1_USB_C
- C4 pad 2: GND_USB -> GND_PWRrt1_USB_C
- C5 pad 1: GND_USB -> GND_PWRrt1_USB_C
- C5 pad 2: VDD -> 3V3_RPi
- C52 pad 1: VDD -> 3V3_RPi
- C52 pad 2: GND_USB -> GND_PWRrt1_USB_C
- C6 pad 1: GND_USB -> GND_PWRrt1_USB_C
- C6 pad 2: VDD -> 3V3_RPi
- C7 pad 1: VDD -> 3V3_RPi
- C7 pad 2: GND_USB -> GND_PWRrt1_USB_C
- C8 pad 1: GND_USB -> GND_PWRrt1_USB_C
- C8 pad 2: VDD -> 3V3_RPi
- C9 pad 1: GND_USB -> GND_PWRrt1_USB_C
- C9 pad 2: VDD -> 3V3_RPi
- D1 pad 1: V+_ISO -> V+_ISO_RAW
- D2 pad 1: V+_ISO -> V+_ISO_RAW
- D4 pad 2: V+ -> VBUS_USB
- J1 pad 1: GND_USB -> 3V3_RPi
- J1 pad 2: VDD -> 3V3_RPi
- J2 pad A1: GND_USB -> GND_PWRrt1_USB_C
- J2 pad A12: GND_USB -> GND_PWRrt2_USB_C
- J2 pad A4: V+ -> 5V_RPi
- J2 pad A6: D+_USB_UART -> D+_USB_C
- J2 pad A7: D-_USB_UART -> D-_USB_C
- J2 pad A9: V+ -> VBUS2_USB_C
- J2 pad B1: GND_USB -> GND_PWRrt1_USB_C
- J2 pad B12: GND_USB -> GND_PWRrt2_USB_C
- J2 pad B4: V+ -> 5V_RPi
- J2 pad B6: D+_USB_UART -> D+_USB_C
- J2 pad B7: D-_USB_UART -> D-_USB_C
- J2 pad B9: V+ -> VBUS2_USB_C
- P6 pad 1: VDD -> VBUS_USB1
- P6 pad 2: UART0_RX_WIFI -> D-_USB1
- P6 pad 3: UART0_CTS_WIFI -> D+_USB1
- P6 pad 4: UART0_TX_WIFI -> ID_USB1
- P6 pad 5: UART0_RTS_WIFI -> GND_USB1
- P6 pad 6: GND_USB -> Net-(P6-Pad6)
- P7 pad 1: VDD -> VBUS_USB2
- P7 pad 2: SPI5_NSS -> D-_USB2
- P7 pad 3: SPI5_SCK -> D+_USB2
- P7 pad 4: SPI5_MOSI -> ID_USB2
- P7 pad 5: SPI5_MISO -> GND_USB2
- P7 pad 6: GND_USB -> Net-(P7-Pad6)
- R2 pad 1: GND_USB -> GND_PWRrt1_USB_C
- R3 pad 2: GND_USB -> GND_PWRrt1_USB_C
- R4 pad 2: GND_USB -> GND_PWRrt1_USB_C
- R5 pad 2: V+ -> 5V_RPi
- R8 pad 1: VDD -> 3V3_RPi
- R9 pad 2: VDD -> 3V3_RPi
- SW1 pad 2: GND_USB -> GND_PWRrt1_USB_C
- SW2 pad 2: VDD -> 3V3_RPi
- SW3 pad 2: GND_USB -> GND_PWRrt1_USB_C
- SW4 pad 2: GND_USB -> GND_PWRrt1_USB_C
- T1 pad 7: AD1_START -> GND_ISO_RAW
- U10 pad 1: VDD -> 3V3_RPi
- U10 pad 11: AD_SI -> AD_SO
- U10 pad 12: AD_SO -> AD_SI
- U10 pad 2: GND_USB -> GND_PWRrt1_USB_C
- U10 pad 3: SPI2_NSS_AD3 -> AD3_CS_ISO
- U10 pad 4: SPI2_SCK -> AD_SCK_ISO
- U10 pad 5: SPI2_MISO -> AD_SI_ISO
- U10 pad 6: SPI2_MOSI -> AD_SO_ISO
- U10 pad 8: GND_USB -> GND_PWRrt1_USB_C
- U11 pad 1: GND_USB -> GND_PWRrt1_USB_C
- U11 pad 2: VDD -> 3V3_RPi
- U11 pad 3: V+ -> 5V_RPi
- U12 pad 1: SPI3_MISO -> SDO_SA0_ACC
- U12 pad 12: SPI3_NSS -> CS_ACC
- U12 pad 13: SPI3_SCK -> I2C1_SCL
- U12 pad 14: SPI3_MOSI -> I2C1_SDA
- U12 pad 2: GND_USB -> GND_PWRrt1_USB_C
- U12 pad 3: GND_USB -> GND_PWRrt1_USB_C
- U12 pad 4: Net-(U12-Pad4) -> INT1_ACC
- U12 pad 5: VDD -> 3V3_RPi
- U12 pad 6: GND_USB -> GND_PWRrt1_USB_C
- U12 pad 7: GND_USB -> GND_PWRrt1_USB_C
- U12 pad 8: VDD -> 3V3_RPi
- U12 pad 9: Net-(U12-Pad9) -> INT2_ACC
- U37 pad 1: SPI1_SCK -> AD1_DCLK_ISO
- U37 pad 10: Net-(U37-Pad10) -> I2C2_SDA
- U37 pad 100: Net-(U37-Pad100) -> MCO1
- U37 pad 102: ID_USB -> USART1_RX
- U37 pad 103: D-_USB -> USB_OTG_FS_DM
- U37 pad 104: D+_USB -> USB_OTG_FS_DP
- U37 pad 105: SWDIO -> SYS_JTMS-SWDIO
- U37 pad 107: GND_USB -> GND_PWRrt1_USB_C
- U37 pad 108: VDD -> 3V3_RPi
- U37 pad 109: SWCLK -> SYS_JTCK-SWCLK
- U37 pad 11: Net-(U37-Pad11) -> I2C2_SCL
- U37 pad 110: SPI3_NSS -> SYS_JTDI
- U37 pad 111: SDIO_D2 -> SDMMC1_D2
- U37 pad 112: SDIO_D3 -> SDMMC1_D3
- U37 pad 113: SDIO_CK -> SDMMC1_CK
- U37 pad 116: SDIO_CMD -> SDMMC1_CMD
- U37 pad 12: Net-(U37-Pad12) -> AD2_CS_ISO
- U37 pad 120: GND_USB -> GND_PWRrt1_USB_C
- U37 pad 121: VDD -> 3V3_RPi
- U37 pad 122: Net-(U37-Pad122) -> CLK_SDIO
- U37 pad 123: Net-(U37-Pad123) -> CMD_SDIO
- U37 pad 124: Net-(U37-Pad124) -> DATA0_SDIO
- U37 pad 125: Net-(U37-Pad125) -> DATA1_SDIO
- U37 pad 126: Net-(U37-Pad126) -> DATA2_SDIO
- U37 pad 127: SPI6_MISO -> DATA3_SDIO
- U37 pad 128: SPI6_SCK -> DETECT_SDIO
- U37 pad 13: Net-(U37-Pad13) -> AD3_CS_ISO
- U37 pad 130: GND_USB -> GND_PWRrt1_USB_C
- U37 pad 131: VDD -> 3V3_RPi
- U37 pad 132: Net-(U37-Pad132) -> INT2_ACC
- U37 pad 133: SPI3_SCK -> SYS_JTDO-SWO
- U37 pad 134: SPI3_MISO -> SYS_JTRST
- U37 pad 135: SPI3_MOSI -> INT1_ACC
- U37 pad 14: Net-(U37-Pad14) -> AD4_CS_ISO
- U37 pad 140: Net-(U37-Pad140) -> AD1_CS_ISO
- U37 pad 143: Net-(U37-Pad143) -> 3V3_RPi
- U37 pad 144: VDD -> 3V3_RPi
- U37 pad 15: Net-(U37-Pad15) -> AD1_RESET_ISO
- U37 pad 16: GND_USB -> GND_PWRrt1_USB_C
- U37 pad 17: VDD -> 3V3_RPi
- U37 pad 18: SPI5_NSS -> Net-(U37-Pad18)
- U37 pad 19: SPI5_SCK -> Net-(U37-Pad19)
- U37 pad 20: SPI5_MISO -> AD1_DCLK_ISO
- U37 pad 21: SPI5_MOSI -> AD1_DRDY_ISO
- U37 pad 27: Net-(U37-Pad27) -> ETH_MDC
- U37 pad 28: Net-(U37-Pad28) -> AD_SO_ISO
- U37 pad 29: Net-(U37-Pad29) -> AD_SI_ISO
- U37 pad 3: SPI4_NSS -> AD1_DOUT0_ISO
- U37 pad 30: VDD -> 3V3_RPi
- U37 pad 31: GND_USB -> GND_PWRrt1_USB_C
- U37 pad 32: VDD -> 3V3_RPi
- U37 pad 33: VDD -> 3V3_RPi
- U37 pad 34: UART0_CTS_WIFI -> AD1_DCLK_ISO
- U37 pad 35: UART0_RTS_WIFI -> ETH_REF_CLK
- U37 pad 36: UART0_TX_WIFI -> ETH_MDIO
- U37 pad 37: UART0_RX_WIFI -> Net-(U37-Pad37)
- U37 pad 38: GND_USB -> GND_PWRrt1_USB_C
- U37 pad 39: VDD -> 3V3_RPi
- U37 pad 40: SPI1_NSS -> SPI6_NSS
- U37 pad 41: SPI1_SCK -> AD1_DCLK_ISO
- U37 pad 42: SPI1_MISO -> SPI6_MISO
- U37 pad 43: SPI1_MOSI -> ETH_CRS_DV
- U37 pad 44: Net-(U37-Pad44) -> ETH_RXD0
- U37 pad 45: Net-(U37-Pad45) -> ETH_RXD1
- U37 pad 51: GND_USB -> GND_PWRrt1_USB_C
- U37 pad 52: VDD -> 3V3_RPi
- U37 pad 54: AD_RESET -> Net-(U37-Pad54)
- U37 pad 58: Net-(U37-Pad58) -> AD1_DCLK_ISO
- U37 pad 6: VDD -> 3V3_RPi
- U37 pad 60: Net-(U37-Pad60) -> AD1_DRDY_ISO
- U37 pad 61: GND_USB -> GND_PWRrt1_USB_C
- U37 pad 62: VDD -> 3V3_RPi
- U37 pad 69: I2C2_SCL -> AD_SCK_ISO
- U37 pad 70: I2C2_SDA -> ETH_TX_EN
- U37 pad 72: VDD -> 3V3_RPi
- U37 pad 73: SPI2_NSS -> ETH_TXD0
- U37 pad 74: SPI2_SCK -> ETH_TXD1
- U37 pad 75: SPI2_MISO -> D-_USB_C
- U37 pad 76: SPI2_MOSI -> D+_USB_C
- U37 pad 77: USART3_TX -> RX_UART_USB
- U37 pad 78: USART3_RX -> TX_UART_USB
- U37 pad 80: USART3_CTS -> RTS_UART_USB
- U37 pad 81: USART3_RTS -> CTS_UART_USB
- U37 pad 83: GND_USB -> GND_PWRrt1_USB_C
- U37 pad 84: VDD -> 3V3_RPi
- U37 pad 93: SPI6_NSS -> Net-(U37-Pad93)
- U37 pad 94: GND_USB -> GND_PWRrt1_USB_C
- U37 pad 95: VDD -> 3V3_RPi
- U37 pad 96: Net-(U37-Pad96) -> AD1_DRDY_ISO
- U37 pad 97: SDIO_DETECT -> Net-(U37-Pad97)
- U37 pad 98: SDIO_D0 -> SDMMC1_D0
- U37 pad 99: SDIO_D1 -> SDMMC1_D1
- U43 pad 1: SDIO_D2 -> DATA2_SDIO
- U43 pad 2: SDIO_D3 -> DATA3_SDIO
- U43 pad 3: SDIO_CMD -> CMD_SDIO
- U43 pad 4: VDD -> 3V3_RPi
- U43 pad 5: SDIO_CK -> CLK_SDIO
- U43 pad 6: GND_USB -> GND_PWRrt1_USB_C
- U43 pad 7: SDIO_D0 -> DATA0_SDIO
- U43 pad 8: SDIO_D1 -> DATA1_SDIO
- U43 pad 9: SDIO_DETECT -> DETECT_SDIO
- U5 pad 11: SPI2_NSS_AD2 -> AD2_CS_ISO
- U5 pad 12: SPI2_NSS -> AD1_CS_ISO
- U5 pad 13: SPI1_SCK -> AD1_DCLK_ISO
- U5 pad 14: SPI1_NSS -> AD1_DRDY_ISO
- U5 pad 15: GND_USB -> GND_PWRrt1_USB_C
- U5 pad 16: VDD -> 3V3_RPi
- U5 pad 9: GND_USB -> GND_PWRrt1_USB_C
- U7 pad 1: GND_USB -> GND_PWRrt1_USB_C
- U7 pad 13: SPI5_SCK -> MTMS
- U7 pad 14: SPI5_MISO -> MTDI
- U7 pad 15: GND_USB -> GND_PWRrt1_USB_C
- U7 pad 16: SPI5_MOSI -> MTCK
- U7 pad 2: VDD -> 3V3_RPi
- U7 pad 23: SPI5_NSS -> MTDO
- U7 pad 31: UART0_CTS_WIFI -> RTS_UART_USB
- U7 pad 32: UART0_RTS_WIFI -> Net-(U7-Pad32)
- U7 pad 34: UART0_RX_WIFI -> TX_UART_USB
- U7 pad 35: UART0_TX_WIFI -> RX_UART_USB
- U7 pad 36: UART0_RTS_WIFI -> CTS_UART_USB
- U7 pad 38: GND_USB -> GND_PWRrt1_USB_C
- U7 pad 39: GND_USB -> GND_PWRrt1_USB_C
- U8 pad 23: UART0_RTS_WIFI -> CTS_UART_USB
- U8 pad 24: UART0_CTS_WIFI -> RTS_UART_USB
- U8 pad 25: UART0_TX_WIFI -> RX_UART_USB
- U8 pad 26: UART0_RX_WIFI -> TX_UART_USB
- U8 pad 29: GND_USB -> GND_PWRrt1_USB_C
- U8 pad 3: GND_USB -> GND_PWRrt1_USB_C
- U8 pad 5: D-_USB_UART -> D+_USB_C_2
- U8 pad 6: VDD -> 3V3_RPi
- U8 pad 7: VDD -> 3V3_RPi
- U9 pad 11: SPI2_NSS_AD4 -> AD4_CS_ISO
- U9 pad 12: AD_RESET -> AD1_RESET_ISO
- U9 pad 14: SPI1_MOSI -> AD1_DOUT0_ISO
- U9 pad 15: GND_USB -> GND_PWRrt1_USB_C
- U9 pad 16: VDD -> 3V3_RPi
- U9 pad 9: GND_USB -> GND_PWRrt1_USB_C
Routing:
- net VDD: track 271.9 -> 0.00 mm, vias 22 -> 0
- net GND_PWRrt1_USB_C: track 0.00 -> 190.9 mm, vias 0 -> 26
- net GND_USB: track 189.7 -> 0.00 mm, vias 28 -> 0
- net 3V3_RPi: track 0.00 -> 149.7 mm, vias 0 -> 24
- net AD1_DRDY_ISO: track 0.00 -> 107.2 mm, vias 0 -> 1
- net AD1_DCLK_ISO: track 0.00 -> 92.1 mm, vias 0 -> 1
- net AD_SCK_ISO: track 0.00 -> 82.9 mm, vias 0 -> 1
- net 5V_RPi: track 0.00 -> 68.5 mm, vias 0 -> 1
- net MTCK: track 0.00 -> 68.4 mm
- net CTS_UART_USB: track 0.00 -> 68.1 mm, vias 0 -> 2
- net V+: track 65.5 -> 0.00 mm, vias 4 -> 0
- net EN_WIFI: track 0.00 -> 64.7 mm, vias 0 -> 2
- net MTDI: track 0.00 -> 62.2 mm
- net GND_RAW: track 10.1 -> 72.3 mm, vias 0 -> 1
- net UART0_RTS_WIFI: track 59.4 -> 0.00 mm, vias 4 -> 0
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- added copper zone on In2.Cu, net 3V3_RPi
- added copper zone on In1.Cu, net GND_RPi
- removed copper zone on In1.Cu, net GND_USB
- removed copper zone on In2.Cu, net V+
- removed copper zone on In2.Cu, net VDD
Other:
- board size 66 x 66 mm -> 66 x 76.2 mm
- board text removed: "AVDD"
- board text removed: "IOVDD"
- board text removed: "V+"
- board text removed: "V+_ISO"
- board text removed: "VDD"
