File: KiCad/FreeEEG32-alpha2.sch (KiCad schematic (older format))
At the start: 66 parts, among them J1 CONN_01X02, P11 CONN_01X03, P6 CONN_02X03, P7 CONN_02X03, SW1 NRST, SW2 BOOT0, U1 ADP7118AUJZ-3.3, U10 ISO7341c_spi, U11 AMS1117-3.3, U12 LSM6DS3, U2 ADP7118AUJZ-3.3, U3 8.192MHz, U37 STM32F427ZI_4side_short, U4 ADR4525, U43 473521001, U5 ADUM1402BRWZ, U9 ADUM1402BRWZ, Y1 32768Hz, Y2 8MHz

Commit message: Add files via upload
Parts:
- removed J1: CONN_01X02, Connector_PinSocket_2.54mm:PinSocket_1x02_P2.54mm_Vertical, symbol Connector_Generic:Conn_01x02
- removed P11: CONN_01X03, Connector_PinSocket_2.54mm:PinSocket_1x03_P2.54mm_Vertical, symbol Connector_Generic:Conn_01x03
- removed P6, P7: CONN_02X03, Connector_PinSocket_2.54mm:PinSocket_2x03_P2.54mm_Vertical, symbol Connector_Generic:Conn_02x03_Odd_Even
- added C139, C140: 100n, Capacitor_SMD:C_0402_1005Metric, symbol Device:C_Small
- added C141, C142: 1u, Capacitor_SMD:C_0402_1005Metric, symbol Device:C_Small
- added J1: Conn_02x07_Odd_Even, Connector_PinSocket_2.54mm:PinSocket_2x07_P2.54mm_Horizontal, symbol Connector_Generic:Conn_02x07_Odd_Even
- added J4: Conn_02x07_Odd_Even, Connector_PinHeader_2.54mm:PinHeader_2x07_P2.54mm_Horizontal, symbol Connector_Generic:Conn_02x07_Odd_Even
- added J6: Conn_02x20_Odd_Even, Connector_PinSocket_2.54mm:PinSocket_2x20_P2.54mm_Vertical, symbol Connector_Generic:Conn_02x20_Odd_Even
- added R10: 0, Resistor_SMD:R_0402_1005Metric, symbol Device:R_Small
- added U14, U15, U16: ISO7341c_spi, Package_SO:SOIC-16W_7.5x10.3mm_P1.27mm, symbol iso7341c:ISO7341c
- added U17: CAT24M01W, Package_SO:SOIC-8_3.9x4.9mm_P1.27mm, symbol Memory_EEPROM:CAT24M01W
- U12: footprint Housings_LGA_FreeEEG32:LGA-14L_2.5x3mm_Pitch0.5mm -> LSM6DS3TR:Bosch_LGA-14_3x2.5mm_P0.5mm
Connections:
- net labels added: 3V3_RPi, 5V_RPi, AD1_CS_ISO, AD1_DCLK_ISO, AD1_DOUT0_ISO, AD1_DOUT1_ISO, AD1_DRDY_ISO, AD1_RESET_ISO, AD2_CS_ISO, AD3_CS_ISO, AD4_CS_ISO, AD_DRDY, AD_SCK_ISO, AD_SI_ISO, AD_SO_ISO, BOOT0, BOOT1, CAN1_RX, CAN1_TX, CLK_SDIO, CMD_SDIO, CS_ACC, DATA0_SDIO, DATA1_SDIO, DATA2_SDIO, DATA3_SDIO, DETECT_SDIO, EN_WIFI, ETH_COL, ETH_CRS_DV, ETH_MDC, ETH_MDIO, ETH_REF_CLK, ETH_RXD0, ETH_RXD1, ETH_TXD0, ETH_TXD1, ETH_TX_EN, GND_RAW, GND_RPi, GND_USB_UART, GPCLK0_RPi, GPCLK1_RPi, GPCLK2_RPi, GPIO_0_RPi, GPIO_25_RPi, GPIO_2_RPi, GPIO_3_RPi, GPIO_4_RPi, GPIO_5_RPi, GPIO_6_RPi, I2C1_SCL, I2C1_SDA, I2S1_CK, I2S1_WS, ID_SC_RPi, ID_SD_RPi, INT1_ACC, INT2_ACC, MCO1, MCO2, MISO0_RPi, MISO1_RPi, MOSI0_RPi, MOSI1_RPi, MTCK, MTDI, MTDO, MTMS, PCM0_CLK_OPi, PCM0_DIN_OPi, PCM0_DOUT_OPi, PCM0_SYNC_OPi, PCM_CLK_RPi, PCM_DIN_RPi, PCM_DOUT_RPi, PCM_FS_RPi, PWM0_RPi, PWM1_RPi, RXD_RPi, SAI1_FS_B, SAI1_SCK_B, SAI1_SD_A, SAI1_SD_B, SAI2_FS_B, SAI2_SCK_B, SAI2_SD_A, SAI2_SD_B, SCL1_RPi, SCLK0_RPi, SCLK1_RPi, SCL_ACC, SDA1_RPi, SDA_ACC, SDMMC1_CK, SDMMC1_CMD, SDMMC1_D0, SDMMC1_D1, SDMMC1_D2, SDMMC1_D3, SDMMC1_DETECT, SDMMC2_CK, SDMMC2_CMD, SDMMC2_D0, SDMMC2_D1, SDMMC2_D2, SDMMC2_D3, SDMMC2_DETECT, SDO_SA0_ACC, SPI0_CE0_RPi, SPI0_CE1_RPi, SPI1_CE0_RPi, SPI1_CE1_RPi, SPI1_CE2_RPi, SYS_JTCK-SWCLK, SYS_JTDI, SYS_JTDO-SWO, SYS_JTMS-SWDIO, SYS_JTRST, TIM1_CH1, TIM1_ETR, TIM8_CH1, TIM8_CH2, TIM8_ETR, TXD_RPi, UART7_RX, UART7_TX, UART8_RX, UART8_TX, USB_OTG_HS_DM, USB_OTG_HS_DP, V+_RAW, VBUS_USB_UART
- net labels removed: SDIO_CK, SDIO_CMD, SDIO_D0, SDIO_D1, SDIO_D2, SDIO_D3, SDIO_DETECT, SPI2_NSS, SPI3_NSS, SPI6_MOSI, SPI6_SCK, SWCLK, SWDIO, USART2_CTS, USART2_RTS, USART2_RX, USART2_TX
- wire segments 601 -> 828
- no-connect marks 83 -> 41
Other:
- moved on the sheet: C107, C108, C125, C128, C129, C130, C131, C24, C25, C42, C52, R2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
