File: KiCad/ISO_WIFI_USB.sch (KiCad schematic (older format))
At the start: 33 parts, among them J2 USB_C_Receptacle, J3 Conn_02x02_Odd_Even, P5 USB_OTG, SW3 RST, SW4 BOOT, T1 da2303, U6 SN6505B, U7 ESP32-WROOM-32, U8 CP2102N-28

Commit message: Add files via upload
Parts:
- removed J2: USB_C_Receptacle, Connector_USB:USB_C_Receptacle_Amphenol_12401610E4-2A_CircularHoles, symbol FreeEEG32-alpha-2-rescue:USB_C_Receptacle-Connector
- added J10, J12, J5, J7, J8, J9: Conn_01x02, Connector_PinHeader_2.54mm:PinHeader_1x02_P2.54mm_Vertical, symbol Connector_Generic:Conn_01x02
- added J11, J2: USB_C_Receptacle-Connector_VBUS2, Connector_USB:USB_C_Receptacle_Amphenol_12401548E4-2A, symbol FreeEEG32-alpha-2-rescue:USB_C_Receptacle-Connector_VBUS2
- added P6, P7, P8: USB_OTG, Connector_USB:USB_Micro-B_Molex-105017-0001, symbol Connector:USB_B_Micro
Connections:
- net labels added: CLK_WIFI, CTS_UART_USB, D+_USB1, D+_USB2, D+_USB_C, D+_USB_C_2, D-_USB1, D-_USB2, D-_USB_C, D-_USB_C_2, EMAC_RXD0, EMAC_RXD1, EMAC_RX_DV, GND_ISO_RAW, GND_PWRrt1_USB_C, GND_PWRrt1_USB_C_2, GND_PWRrt2_USB_C, GND_PWRrt2_USB_C_2, GND_USB1, GND_USB2, GPIO0_WIFI, GPIO2_WIFI, HSPICLK_WIFI, HSPICS0_WIFI, HSPID_WIFI, HSPIQ_WIFI, ID_USB1, ID_USB2, MTCK, MTDI, MTDO, MTMS, RTS_UART_USB, RX_UART_USB, TX_UART_USB, U0CTS_WIFI, U0RTS_WIFI, U0RXD_WIFI, U0TXD_WIFI, U1CTS_WIFI, U1RTS_WIFI, U1RXD_WIFI, U1TXD_WIFI, USART1_CTS, USART1_RTS, USART1_RX, USART1_TX, USART3_CTS, USART3_RTS, USART3_RX, USART3_TX, USB_OTG_HS_DM, USB_OTG_HS_DP, V+_ISO_RAW, VBUS1_USB_C, VBUS1_USB_C_2, VBUS2_USB_C, VBUS2_USB_C_2, VBUS_USB1, VBUS_USB2, VDD_USB_UART, VSPICLK_WIFI, VSPICS0_WIFI, VSPID_WIFI, VSPIQ_WIFI
- net labels removed: IO0_WIFI, SPI5_MISO, SPI5_MOSI, SPI5_NSS, SPI5_SCK, UART0_CTS_WIFI, UART0_RTS_WIFI, UART0_RX_WIFI, UART0_TX_WIFI, UART_CTS_USB, UART_RTS_USB, UART_RX_USB, UART_TX_USB
- wire segments 163 -> 242
- no-connect marks 53 -> 61
Other:
- moved on the sheet: C113, C114, C115, C132, C134, D1, D2, D3, D4, H1, H2, H3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
